File: Schematics/esquema_electronica_final/_autosave-schematics.kicad_sch (KiCad schematic)
At the start: 28 parts, among them SW1 POWER_SWITCH, U1 ESP32-S3-DEVKITC-1-N16R8

Commit message: last kicad schematic
Parts:
- added BATTERY: ~, symbol mario:BATERIA
Connections:
- net at F1.1: now also BATTERY. (GND)
- new net: MOTOR_BRUSHLESS_RIGHT. (H_GND), ZS-X11_RIGHT. (ANALOG_CTRL) (x3)
- new net: MOTOR_BRUSHLESS_LEFT. (H_GND), ZS-X11_LEFT. (ANALOG_CTRL) (x3)
- new net: BATTERY. (GND), SEN0291. (GND)
Changed lines of the file:
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@@
 	(wire
 		(pts
-			(xy 30.48 26.67) (xy 38.1 26.67)
+			(xy 34.29 26.67) (xy 38.1 26.67)
 		)
 		(stroke
@@
 	(wire
 		(pts
-			(xy 30.48 29.21) (xy 35.56 29.21)
+			(xy 34.29 29.21) (xy 35.56 29.21)
 		)
 		(stroke
@@
 					(unit 1)
 				)
+			)
+		)
+	)
+	(symbol
+		(lib_id "mario:BATERIA")
+		(at 25.4 22.86 0)
+		(unit 1)
+		(exclude_from_sim no)
+		(in_bom yes)
+		(on_board yes)
+		(dnp no)
+		(property "Reference" "BATTERY"
+			(at 25.4 33.274 0)
+			(effects
+				(font
+					(size 1.27 1.27)
+				)
+			)
+		)
+		(property "Value" "~"
+			(at 25.4 22.86 0)
+			(effects
+				(font
+					(size 1.27 1.27)
+				)
+			)
+		)
+		(property "Footprint" ""
+			(at 25.4 22.86 0)
+			(effects
+				(font
+					(size 1.27 1.27)
+				)
+				(hide yes)
+			)
+		)
+		(property "Datasheet" ""
+			(at 25.4 22.86 0)
+			(effects
+				(font
+					(size 1.27 1.27)
+				)
+				(hide yes)
+			)
+		)
+		(property "Description" ""
+			(at 25.4 22.86 0)
+			(effects
+				(font
+					(size 1.27 1.27)
+				)
+				(hide yes)
+			)
+		)
+		(pin ""
+		)
+		(pin ""
+		)
+		(instances
+			(project ""
+				(path "/29c96457-b859-4d59-aaa2-52833e6eb6f5"
+					(reference "BATTERY")
+					(unit 1)
+				)
